File: telemetry-lights.kicad_sch (KiCad schematic)
At the start: 27 parts, among them J1 CONN HEADER VERT 3POS 2.5MM, J2 CONN HEADER VERT 4POS 2.5MM, J6 CONN HEADER VERT 2POS 1.5MM, J7 CONN HEADER VERT 2POS 1.5MM, U2 STM32L431KBU6TR, U3 IAM-20381HT

Commit message: minor revisions
Parts:
- added D1: DIODE SCHOTTKY 30V 1A SOD323F, footprints:P39_SOD-323P, symbol symbols:SDB13HS-AQ
- added J5: PIN HEADER 2.54MM PITCH STR DIP, footprints:CONN6x1_G800W302018EU_AMP, symbol symbols:G800W302018EU
Connections:
- net +3.3V is gone; now on net 3V3: C19.1, U3.1 (VDDIO)
- net 3V3: now also D1.1 (K)
- net GND: now also J5.3
- net NRST: now also J5.5
- new net: D1.2 (A), J5.1
- new net SWCLK: J5.2
- new net SWDIO: J5.4
- new net SWO: J5.6
Other:
- note added: "STLink"
- moved on the sheet: BOOT1, C16, C17, C18, C19, C20, C22, C23, C25, C26, C27, C28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

Commit message: Change pin connected to lights
Connections:
- net LIGHT: now also U2.11 (PA5); no longer U2.13 (PA7)
Changed lines of the file:
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@@
+	)
+	(no_connect
+		(at 54.61 63.5)
 	)
 	(no_connect
@@
 	)
 	(no_connect
-		(at 54.61 58.42)
-	)
-	(no_connect
 		(at 54.61 73.66)
 	)
@@
 	(wire
 		(pts
-			(xy 52.07 63.5) (xy 54.61 63.5)
-		)
-		(stroke
-			(width 0)
-			(type default)
-		)
-	)
-	(wire
-		(pts
 			(xy 170.18 162.56) (xy 170.18 165.1)
 		)
@@
 		(pts
 			(xy 274.32 158.75) (xy 274.32 107.95)
+		)
+		(stroke
+			(width 0)
+			(type default)
+		)
+	)
+	(wire
+		(pts
+			(xy 52.07 58.42) (xy 54.61 58.42)
 		)
 		(stroke
@@
 	)
 	(label "LIGHT"
-		(at 52.07 63.5 180)
-		(effects
-			(font
+		(at 52.07 58.42 180)
+		(effects
+			(font

Commit message: second pcb layout
Parts:
- D1: footprint footprints:P39_SOD-323P -> Diode_SMD:D_SOD-323F
- J5: footprint footprints:CONN6x1_G800W302018EU_AMP -> Connector_PinHeader_2.54mm:PinHeader_1x06_P2.54mm_Vertical
Changed lines of the file:
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@@
 			)
 		)
-		(property "Footprint" "footprints:P39_SOD-323P"
+		(property "Footprint" "Diode_SMD:D_SOD-323F"
 			(at 69.215 220.98 0)
 			(hide yes)
@@
 			)
 		)
-		(property "Footprint" "footprints:CONN6x1_G800W302018EU_AMP"
+		(property "Footprint" "Connector_PinHeader_2.54mm:PinHeader_1x06_P2.54mm_Vertical"
 			(at 78.74 227.33 0)
 			(hide yes)
