File: telemetry-lights.kicad_pcb (KiCad board)
At the start: 2 copper layers, 28.8 x 25.5 mm, 29 parts, among them J1 CONN HEADER VERT 3POS 2.5MM, J2 CONN HEADER VERT 4POS 2.5MM, J5 PIN HEADER 2.54MM PITCH STR D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, J7 CONN HEADER VERT 2POS 1.5MM, U2 STM32L431KBU6TR, U3 IAM-20381HT

Commit message: final layout changes
Parts:
- added H1: MountingHole, MountingHole:MountingHole_2.5mm, F.Cu at (101.3, 94.8)
- added H2: MountingHole, MountingHole:MountingHole_2.5mm, F.Cu at (101.4, 114.8)
- D1: footprint skateboard-footprint-library:P39_SOD-323P -> footprints:P39_SOD-323P
- J5: footprint skateboard-footprint-library:CONN6x1_G800W302018EU_AMP -> footprints:CONN6x1_G800W302018EU_AMP
- R5: moved to B.Cu
- moved C20 5.00 mm to (81.5, 97.9), turned to 90 degrees
- moved J2 4.08 mm to (102.0, 100.9)
- moved R1 3.35 mm to (86.1, 97.2), turned to 180 degrees
- moved J6 3.12 mm to (78.5, 115.3)
- moved J1 1.74 mm to (84.8, 113.5)
- moved R2 1.28 mm to (83.4, 97.9), turned to 90 degrees
- moved D1 1.19 mm to (95.2, 97.8), turned to 0 degrees
- moved J5 1.00 mm to (95.4, 93.5)
- moved B 0.60 mm to (86.6, 99.0)
- renumbered 5V to J6
Routing:
- net /SDA: track 22.1 -> 26.5 mm
- net /SCL: track 24.1 -> 27.8 mm
- net Net-(J1-Pad2): track 5.99 -> 7.59 mm
- net 3V3: track 34.2 -> 32.8 mm, vias 4 -> 3
- net /SWDIO: track 8.86 -> 10.2 mm
- net Net-(D1-A): track 3.56 -> 4.90 mm, vias 1 -> 0
- net 5V: track 5.69 -> 7.02 mm
- net GND: track 11.6 -> 12.9 mm, vias 13 -> 18
- net /SWCLK: track 11.4 -> 12.4 mm
- net /NRST: track 14.6 -> 13.8 mm
- net /SWO: track 7.20 -> 7.98 mm
Other:
- board size 28.8 x 25.5 mm -> 31.5 x 26.6 mm
- board text added: "5V"
